File: Advanced_power_control/APC/APC.sch (KiCad schematic (older format))
At the start: 50 parts, among them J1 AVR-JTAG-10, J10 CMD_IN, J11 PWR_V_SEL, J12 12/24 V_IN, J13 220_OUT, J2 EM_STOP_INT, J3 STATUS_LED, J4 EM_STOP, J5 POWER_BUTTON, J6 POWER_LED, J7 220 IN, J8 CMD_OUT, J9 CMD_V_SEL, K1 G5LE-1, Q1 IRLML0030, Q2 IRLML0030, Q3 IRLML0030, U1 ATmega164PA-AU, U2 LTV-817, U3 LTV-817, U4 LTV-817

Commit message: update schematic and board
Parts:
- added C6: 0.1uF, Capacitor_SMD:C_0805_2012Metric_Pad1.15x1.40mm_HandSolder, symbol Device:C_Small
- C1, C2, C3, C4, C5: footprint Capacitor_SMD:C_0805_2012Metric_Pad1.18x1.45mm_HandSolder -> Capacitor_SMD:C_0805_2012Metric_Pad1.15x1.40mm_HandSolder
- C7: renamed from C6; footprint Capacitor_SMD:C_0805_2012Metric_Pad1.18x1.45mm_HandSolder -> Capacitor_SMD:C_0805_2012Metric_Pad1.15x1.40mm_HandSolder
- C8: renamed from C7; footprint Capacitor_SMD:C_0805_2012Metric_Pad1.18x1.45mm_HandSolder -> Capacitor_SMD:C_0805_2012Metric_Pad1.15x1.40mm_HandSolder
- renumbered C8 to C9
Connections:
- net +5V: now also C6.2
- net CMD_IN: now also U1.37 (PA0); no longer U1.43 (PB3)
- net CMD_OUT: now also U1.44 (PB4); no longer U1.34 (PA3)
- net GND: now also C6.1
- net PWR: now also U1.1 (PB5); no longer U1.35 (PA2)
- net STATE: now also U1.3 (PB7); no longer U1.37 (PA0)
- net S_STATE: now also U1.2 (PB6); no longer U1.36 (PA1)
Changed lines of the file:
@@
 $EndComp
 $Comp
-L Device:C_Small C7
+L Device:C_Small C8
 U 1 1 608B60AA
 P 7000 5200
-F 0 "C7" H 6909 5154 50  0000 R CNN
+F 0 "C8" H 6909 5154 50  0000 R CNN
 F 1 "0.01uF" H 6909 5245 50  0000 R CNN
-F 2 "Capacitor_SMD:C_0805_2012Metric_Pad1.18x1.45mm_HandSolder" H 7000 5200 50  0001 C CNN
+F 2 "Capacitor_SMD:C_0805_2012Metric_Pad1.15x1.40mm_HandSolder" H 7000 5200 50  0001 C CNN
 F 3 "~" H 7000 5200 50  0001 C CNN
 	1    7000 5200
@@
 $EndComp
 $Comp
-L Device:C_Small C6
+L Device:C_Small C7
 U 1 1 608C7288
 P 7000 3950
-F 0 "C6" H 6909 3904 50  0000 R CNN
+F 0 "C7" H 6909 3904 50  0000 R CNN
 F 1 "0.01uF" H 6909 3995 50  0000 R CNN
-F 2 "Capacitor_SMD:C_0805_2012Metric_Pad1.18x1.45mm_HandSolder" H 7000 3950 50  0001 C CNN
+F 2 "Capacitor_SMD:C_0805_2012Metric_Pad1.15x1.40mm_HandSolder" H 7000 3950 50  0001 C CNN
 F 3 "~" H 7000 3950 50  0001 C CNN
 	1    7000 3950
@@
 F 0 "C4" H 2659 2854 50  0000 R CNN
 F 1 "0.01uF" H 2659 2945 50  0000 R CNN
-F 2 "Capacitor_SMD:C_0805_2012Metric_Pad1.18x1.45mm_HandSolder" H 2750 2900 50  0001 C CNN
+F 2 "Capacitor_SMD:C_0805_2012Metric_Pad1.15x1.40mm_HandSolder" H 2750 2900 50  0001 C CNN
 F 3 "~" H 2750 2900 50  0001 C CNN
 	1    2750 2900
@@
 F 0 "C5" H 3159 2854 50  0000 R CNN
 F 1 "0.1uF" H 3159 2945 50  0000 R CNN
-F 2 "Capacitor_SMD:C_0805_2012Metric_Pad1.18x1.45mm_HandSolder" H 3250 2900 50  0001 C CNN
+F 2 "Capacitor_SMD:C_0805_2012Metric_Pad1.15x1.40mm_HandSolder" H 3250 2900 50  0001 C CNN
 F 3 "~" H 3250 2900 50  0001 C CNN
 	1    3250 2900
@@
 F 0 "C3" H 2359 2854 50  0000 R CNN
 F 1 "0.1uF" H 2359 2945 50  0000 R CNN
-F 2 "Capacitor_SMD:C_0805_2012Metric_Pad1.18x1.45mm_HandSolder" H 2450 2900 50  0001 C CNN
+F 2 "Capacitor_SMD:C_0805_2012Metric_Pad1.15x1.40mm_HandSolder" H 2450 2900 50  0001 C CNN
 F 3 "~" H 2450 2900 50  0001 C CNN
 	1    2450 2900
@@
 F 0 "C1" H 1759 3554 50  0000 R CNN
 F 1 "0.01uF" H 1759 3645 50  0000 R CNN
-F 2 "Capacitor_SMD:C_0805_2012Metric_Pad1.18x1.45mm_HandSolder" H 1850 3600 50  0001 C CNN
+F 2 "Capacitor_SMD:C_0805_2012Metric_Pad1.15x1.40mm_HandSolder" H 1850 3600 50  0001 C CNN
 F 3 "~" H 1850 3600 50  0001 C CNN
 	1    1850 3600
@@
 F 0 "C2" H 1759 4154 50  0000 R CNN
 F 1 "0.01uF" H 1759 4245 50  0000 R CNN
-F 2 "Capacitor_SMD:C_0805_2012Metric_Pad1.18x1.45mm_HandSolder" H 1850 4200 50  0001 C CNN
+F 2 "Capacitor_SMD:C_0805_2012Metric_Pad1.15x1.40mm_HandSolder" H 1850 4200 50  0001 C CNN
 F 3 "~" H 1850 4200 50  0001 C CNN
 	1    1850 4200
@@
 Text Label 3450 5450 0    50   ~ 0
 TCK
-Text Label 3450 3450 0    50   ~ 0
+Text Label 3450 5050 0    50   ~ 0
 STATE
-Text Label 3450 3550 0    50   ~ 0
+Text Label 3450 4950 0    50   ~ 0
 S_STATE
-Text Label 3450 3650 0    50   ~ 0
+Text Label 3450 4850 0    50   ~ 0
 PWR
-Text Label 3450 3750 0    50   ~ 0
+Text Label 3450 4750 0    50   ~ 0
 CMD_OUT
 Text Label 3450 6850 0    50   ~ 0
@@
 Text Label 3450 6650 0    50   ~ 0
 V_IN_DET
-Text Label 3450 4650 0    50   ~ 0
+Text Label 3450 3450 0    50   ~ 0
 CMD_IN
 $Comp
-L Device:CP_Small C8
+L Device:CP_Small C9
 U 1 1 608AF908
 P 10950 1100
-F 0 "C8" H 10862 1146 50  0000 R CNN
+F 0 "C9" H 10862 1146 50  0000 R CNN
 F 1 "10uF 16V" H 10862 1055 50  0000 R CNN
 F 2 "Capacitor_Tantalum_SMD:CP_EIA-3528-21_Kemet-B_Pad1.50x2.35mm_HandSolder" H 10950 1100 50  0001 C CNN
@@
 	10950 1200 10800 1200
 Connection ~ 10800 1200
+$Comp
+L Device:C_Small C6
+U 1 1 608B998F
+P 3500 2900
+F 0 "C6" H 3409 2854 50  0000 R CNN
+F 1 "0.1uF" H 3409 2945 50  0000 R CNN
+F 2 "Capacitor_SMD:C_0805_2012Metric_Pad1.15x1.40mm_HandSolder" H 3500 2900 50  0001 C CNN
+F 3 "~" H 3500 2900 50  0001 C CNN
+	1    3500 2900
+	1    0    0    1
+$EndComp
+Wire Wire Line
+	3500 2800 3250 2800
+Wire Wire Line
+	3500 3000 3250 3000
+Connection ~ 3250 3000
 $EndSCHEMATC

Commit message: minimize pcb size
Parts:
- J1: footprint Connector_IDC:IDC-Header_2x05_P2.54mm_Vertical -> Connector_PinHeader_2.54mm:PinHeader_2x05_P2.54mm_Vertical
Changed lines of the file:
@@
 F 0 "J1" H 1320 1496 50  0000 R CNN
 F 1 "AVR-JTAG-10" H 1320 1405 50  0000 R CNN
-F 2 "Connector_IDC:IDC-Header_2x05_P2.54mm_Vertical" V 1600 1600 50  0001 C CNN
+F 2 "Connector_PinHeader_2.54mm:PinHeader_2x05_P2.54mm_Vertical" V 1600 1600 50  0001 C CNN
 F 3 " ~" H 475 900 50  0001 C CNN
 	1    1750 1450
